File: kicad/xiao_256.kicad_sch (KiCad schematic)
At the start: 64 parts, among them J1 Conn_01x02_Pin, J2 Conn_01x02_Pin, SW1 GateronLP, SW10 GateronLP, SW11 GateronLP, SW12 GateronLP, SW13 GateronLP, SW14 GateronLP, SW15 GateronLP, SW16 GateronLP, SW17 GateronLP, SW18 GateronLP, SW19 GateronLP, SW2 GateronLP, SW20 GateronLP, SW21 GateronLP, SW22 GateronLP, SW23 GateronLP, SW24 GateronLP, SW25 GateronLP, SW26 GateronLP, SW27 GateronLP, SW28 GateronLP, SW29 GateronLP, SW3 GateronLP, SW30 GateronLP, SW4 GateronLP, SW5 GateronLP, SW6 GateronLP, SW7 GateronLP, SW8 GateronLP, SW9 GateronLP, U1 Seeed XIAO, U2 SK12D07VG4

Commit message: finish routing
Parts:
- added H1, H2, H3, H4, H5, H6: Hole_Pad, xiao_256:Mount_M2, symbol xiao_256:Hole_Pad
Connections:
- no-connect marks 2 -> 8
Changed lines of the file:
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@@
   )
   (no_connect (at 157.48 73.66))
+  (no_connect (at 31.75 146.05))
+  (no_connect (at 62.23 146.05))
   (no_connect (at 215.9 25.4))
+  (no_connect (at 46.99 146.05))
+  (no_connect (at 46.99 137.16))
+  (no_connect (at 62.23 137.16))
+  (no_connect (at 31.75 137.16))
   (wire (pts (xy 215.9 27.94) (xy 219.71 27.94))
     (stroke (width 0) (type default))
@@
     )
   )
+  (symbol (lib_id "xiao_256:Hole_Pad") (at 46.99 143.51 0) (unit 1)
+    (in_bom yes) (on_board yes) (dnp no) (fields_autoplaced)
+    (property "Reference" "H5" (at 49.53 141.605 0)
+      (effects (font (size 1.27 1.27)) (justify left))
+    )
+    (property "Value" "Hole_Pad" (at 49.53 144.145 0)
+      (effects (font (size 1.27 1.27)) (justify left))
+    )
+    (property "Footprint" "xiao_256:Mount_M2" (at 46.99 143.51 0)
+      (effects (font (size 1.27 1.27)) hide)
+    )
+    (property "Datasheet" "" (at 46.99 143.51 0)
+      (effects (font (size 1.27 1.27)) hide)
+    )
+    (pin "1")
+    (instances
+      (project "xiao_256"
+        (path "/5c69b9b2-9a9b-4f27-a098-371b0fd22f6c"
+          (reference "H5") (unit 1)
+        )
+      )
+    )
+  )
   (symbol (lib_id "xiao_256:D") (at 62.23 93.98 90) (unit 1)
     (in_bom yes) (on_board yes) (dnp no) (fields_autoplaced)
@@
     )
   )
+  (symbol (lib_id "xiao_256:Hole_Pad") (at 31.75 143.51 0) (unit 1)
+    (in_bom yes) (on_board yes) (dnp no) (fields_autoplaced)
+    (property "Reference" "H4" (at 34.29 141.605 0)
+      (effects (font (size 1.27 1.27)) (justify left))
+    )
+    (property "Value" "Hole_Pad" (at 34.29 144.145 0)
+      (effects (font (size 1.27 1.27)) (justify left))
+    )
+    (property "Footprint" "xiao_256:Mount_M2" (at 31.75 143.51 0)
+      (effects (font (size 1.27 1.27)) hide)
+    )
+    (property "Datasheet" "" (at 31.75 143.51 0)
+      (effects (font (size 1.27 1.27)) hide)
+    )
+    (pin "1")
+    (instances
+      (project "xiao_256"
+        (path "/5c69b9b2-9a9b-4f27-a098-371b0fd22f6c"
+          (reference "H4") (unit 1)
+        )
+      )
+    )
+  )
   (symbol (lib_id "xiao_256:D") (at 31.75 93.98 90) (unit 1)
     (in_bom yes) (on_board yes) (dnp no) (fields_autoplaced)
@@
     )
   )
+  (symbol (lib_id "xiao_256:Hole_Pad") (at 31.75 134.62 0) (unit 1)
+    (in_bom yes) (on_board yes) (dnp no) (fields_autoplaced)
+    (property "Reference" "H1" (at 34.29 132.715 0)
+      (effects (font (size 1.27 1.27)) (justify left))
+    )
+    (property "Value" "Hole_Pad" (at 34.29 135.255 0)
+      (effects (font (size 1.27 1.27)) (justify left))
+    )
+    (property "Footprint" "xiao_256:Mount_M2" (at 31.75 134.62 0)
+      (effects (font (size 1.27 1.27)) hide)
+    )
+    (property "Datasheet" "" (at 31.75 134.62 0)
+      (effects (font (size 1.27 1.27)) hide)
+    )
+    (pin "1")
+    (instances
+      (project "xiao_256"
+        (path "/5c69b9b2-9a9b-4f27-a098-371b0fd22f6c"
+          (reference "H1") (unit 1)
+        )
+      )
+    )
+  )
   (symbol (lib_id "xiao_256:GateronLP") (at 93.98 106.68 0) (unit 1)
     (in_bom yes) (on_board yes) (dnp no) (fields_autoplaced)
@@
     )
   )
+  (symbol (lib_id "xiao_256:Hole_Pad") (at 46.99 134.62 0) (unit 1)
+    (in_bom yes) (on_board yes) (dnp no) (fields_autoplaced)
+    (property "Reference" "H2" (at 49.53 132.715 0)
+      (effects (font (size 1.27 1.27)) (justify left))
+    )
+    (property "Value" "Hole_Pad" (at 49.53 135.255 0)
+      (effects (font (size 1.27 1.27)) (justify left))
+    )
+    (property "Footprint" "xiao_256:Mount_M2" (at 46.99 134.62 0)
+      (effects (font (size 1.27 1.27)) hide)
+    )
+    (property "Datasheet" "" (at 46.99 134.62 0)
+      (effects (font (size 1.27 1.27)) hide)
+    )
+    (pin "1")
+    (instances
+      (project "xiao_256"
+        (path "/5c69b9b2-9a9b-4f27-a098-371b0fd22f6c"
+          (reference "H2") (unit 1)
+        )
+      )
+    )
+  )
   (symbol (lib_id "xiao_256:GateronLP") (at 33.02 87.63 0) (unit 1)
     (in_bom yes) (on_board yes) (dnp no) (fields_autoplaced)
@@
         (path "/5c69b9b2-9a9b-4f27-a098-371b0fd22f6c"
           (reference "D13") (unit 1)
+        )
+      )
+    )
+  )
+  (symbol (lib_id "xiao_256:Hole_Pad") (at 62.23 143.51 0) (unit 1)
+    (in_bom yes) (on_board yes) (dnp no) (fields_autoplaced)
+    (property "Reference" "H6" (at 64.77 141.605 0)
+      (effects (font (size 1.27 1.27)) (justify left))
+    )
+    (property "Value" "Hole_Pad" (at 64.77 144.145 0)
+      (effects (font (size 1.27 1.27)) (justify left))
+    )
+    (property "Footprint" "xiao_256:Mount_M2" (at 62.23 143.51 0)
+      (effects (font (size 1.27 1.27)) hide)
+    )
+    (property "Datasheet" "" (at 62.23 143.51 0)
+      (effects (font (size 1.27 1.27)) hide)
+    )
+    (pin "1")
+    (instances
+      (project "xiao_256"
+        (path "/5c69b9b2-9a9b-4f27-a098-371b0fd22f6c"
+          (reference "H6") (unit 1)
         )
       )
@@
         )
       )
+    )
+  )
+  (symbol (lib_id "xiao_256:Hole_Pad") (at 62.23 134.62 0) (unit 1)
+    (in_bom yes) (on_board yes) (dnp no) (fields_autoplaced)
+    (property "Reference" "H3" (at 64.77 132.715 0)
+      (effects (font (size 1.27 1.27)) (justify left))
+    )
+    (property "Value" "Hole_Pad" (at 64.77 135.255 0)
+      (effects (font (size 1.27 1.27)) (justify left))
+    )
+    (property "Footprint" "xiao_256:Mount_M2" (at 62.23 134.62 0)
+      (effects (font (size 1.27 1.27)) hide)
+    )
+    (property "Datasheet" "" (at 62.23 134.62 0)
+      (effects (font (size 1.27 1.27)) hide)
+    )
+    (pin "1")
+    (instances
+      (project "xiao_256"
+        (path "/5c69b9b2-9a9b-4f27-a098-371b0fd22f6c"
+          (reference "H3") (unit 1)
+        )
+      )

Commit message: add cover, tweak footprints
Parts:
- D1, D10, D11, D12, D13, D14, D15, D16, D17, D18, D19, D2, D20, D21, D22, D23, D24, D25, D26, D27, D28, D29, D3, D30, D4, D5, D6, D7, D8, D9: footprint Diode_THT:D_DO-35_SOD27_P7.62mm_Horizontal -> xiao_256:D_DO-35_SOD27_P7.62mm_Horizontal
- J1, J2: footprint Connector_PinHeader_2.54mm:PinHeader_1x02_P2.54mm_Vertical -> xiao_256:PinHeader_1x02_P2.54mm_Vertical
Changed lines of the file:
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@@
       (effects (font (size 1.27 1.27)) (justify right))
     )
-    (property "Footprint" "Diode_THT:D_DO-35_SOD27_P7.62mm_Horizontal" (at 46.99 55.88 90)
+    (property "Footprint" "xiao_256:D_DO-35_SOD27_P7.62mm_Horizontal" (at 46.99 55.88 90)
       (effects (font (size 1.27 1.27)) hide)
     )
@@
       (effects (font (size 1.27 1.27)) (justify right))
     )
-    (property "Footprint" "Diode_THT:D_DO-35_SOD27_P7.62mm_Horizontal" (at 107.95 55.88 90)
+    (property "Footprint" "xiao_256:D_DO-35_SOD27_P7.62mm_Horizontal" (at 107.95 55.88 90)
       (effects (font (size 1.27 1.27)) hide)
     )
@@
       (effects (font (size 1.27 1.27)) (justify right))
     )
-    (property "Footprint" "Diode_THT:D_DO-35_SOD27_P7.62mm_Horizontal" (at 62.23 113.03 90)
+    (property "Footprint" "xiao_256:D_DO-35_SOD27_P7.62mm_Horizontal" (at 62.23 113.03 90)
       (effects (font (size 1.27 1.27)) hide)
     )
@@
       (effects (font (size 1.27 1.27)) (justify right))
     )
-    (property "Footprint" "Diode_THT:D_DO-35_SOD27_P7.62mm_Horizontal" (at 46.99 36.83 90)
+    (property "Footprint" "xiao_256:D_DO-35_SOD27_P7.62mm_Horizontal" (at 46.99 36.83 90)
       (effects (font (size 1.27 1.27)) hide)
     )
@@
       (effects (font (size 1.27 1.27)) (justify right))
     )
-    (property "Footprint" "Diode_THT:D_DO-35_SOD27_P7.62mm_Horizontal" (at 92.71 113.03 90)
+    (property "Footprint" "xiao_256:D_DO-35_SOD27_P7.62mm_Horizontal" (at 92.71 113.03 90)
       (effects (font (size 1.27 1.27)) hide)
     )
@@
       (effects (font (size 1.27 1.27)) (justify right))
     )
-    (property "Footprint" "Diode_THT:D_DO-35_SOD27_P7.62mm_Horizontal" (at 92.71 93.98 90)
+    (property "Footprint" "xiao_256:D_DO-35_SOD27_P7.62mm_Horizontal" (at 92.71 93.98 90)
       (effects (font (size 1.27 1.27)) hide)
     )
@@
       (effects (font (size 1.27 1.27)) (justify right))
     )
-    (property "Footprint" "Diode_THT:D_DO-35_SOD27_P7.62mm_Horizontal" (at 46.99 74.93 90)
+    (property "Footprint" "xiao_256:D_DO-35_SOD27_P7.62mm_Horizontal" (at 46.99 74.93 90)
       (effects (font (size 1.27 1.27)) hide)
     )
@@
       (effects (font (size 1.27 1.27)) (justify right))
     )
-    (property "Footprint" "Diode_THT:D_DO-35_SOD27_P7.62mm_Horizontal" (at 46.99 93.98 90)
+    (property "Footprint" "xiao_256:D_DO-35_SOD27_P7.62mm_Horizontal" (at 46.99 93.98 90)
       (effects (font (size 1.27 1.27)) hide)
     )
@@
       (effects (font (size 1.27 1.27)) (justify right))
     )
-    (property "Footprint" "Diode_THT:D_DO-35_SOD27_P7.62mm_Horizontal" (at 31.75 36.83 90)
+    (property "Footprint" "xiao_256:D_DO-35_SOD27_P7.62mm_Horizontal" (at 31.75 36.83 90)
       (effects (font (size 1.27 1.27)) hide)
     )
@@
       (effects (font (size 1.27 1.27)) (justify right))
     )
-    (property "Footprint" "Diode_THT:D_DO-35_SOD27_P7.62mm_Horizontal" (at 92.71 74.93 90)
+    (property "Footprint" "xiao_256:D_DO-35_SOD27_P7.62mm_Horizontal" (at 92.71 74.93 90)
       (effects (font (size 1.27 1.27)) hide)
     )
@@
       (effects (font (size 1.27 1.27)) (justify right))
     )
-    (property "Footprint" "Diode_THT:D_DO-35_SOD27_P7.62mm_Horizontal" (at 62.23 55.88 90)
+    (property "Footprint" "xiao_256:D_DO-35_SOD27_P7.62mm_Horizontal" (at 62.23 55.88 90)
       (effects (font (size 1.27 1.27)) hide)
     )
@@
       (effects (font (size 1.27 1.27)) (justify right))
     )
-    (property "Footprint" "Diode_THT:D_DO-35_SOD27_P7.62mm_Horizontal" (at 62.23 93.98 90)
+    (property "Footprint" "xiao_256:D_DO-35_SOD27_P7.62mm_Horizontal" (at 62.23 93.98 90)
       (effects (font (size 1.27 1.27)) hide)
     )
@@
       (effects (font (size 1.27 1.27)) (justify right))
     )
-    (property "Footprint" "Diode_THT:D_DO-35_SOD27_P7.62mm_Horizontal" (at 62.23 74.93 90)
+    (property "Footprint" "xiao_256:D_DO-35_SOD27_P7.62mm_Horizontal" (at 62.23 74.93 90)
       (effects (font (size 1.27 1.27)) hide)
     )
@@
       (effects (font (size 1.27 1.27)))
     )
-    (property "Footprint" "Connector_PinHeader_2.54mm:PinHeader_1x02_P2.54mm_Vertical" (at 200.66 77.47 0)
+    (property "Footprint" "xiao_256:PinHeader_1x02_P2.54mm_Vertical" (at 200.66 77.47 0)
       (effects (font (size 1.27 1.27)) hide)
     )
@@
       (effects (font (size 1.27 1.27)) (justify right))
     )
-    (property "Footprint" "Diode_THT:D_DO-35_SOD27_P7.62mm_Horizontal" (at 46.99 113.03 90)
+    (property "Footprint" "xiao_256:D_DO-35_SOD27_P7.62mm_Horizontal" (at 46.99 113.03 90)
       (effects (font (size 1.27 1.27)) hide)
     )
@@
       (effects (font (size 1.27 1.27)))
     )
-    (property "Footprint" "Connector_PinHeader_2.54mm:PinHeader_1x02_P2.54mm_Vertical" (at 200.66 66.04 0)
+    (property "Footprint" "xiao_256:PinHeader_1x02_P2.54mm_Vertical" (at 200.66 66.04 0)
       (effects (font (size 1.27 1.27)) hide)
     )
@@
       (effects (font (size 1.27 1.27)) (justify right))
     )
-    (property "Footprint" "Diode_THT:D_DO-35_SOD27_P7.62mm_Horizontal" (at 77.47 93.98 90)
+    (property "Footprint" "xiao_256:D_DO-35_SOD27_P7.62mm_Horizontal" (at 77.47 93.98 90)
       (effects (font (size 1.27 1.27)) hide)
     )
@@
       (effects (font (size 1.27 1.27)) (justify right))
     )
-    (property "Footprint" "Diode_THT:D_DO-35_SOD27_P7.62mm_Horizontal" (at 77.47 36.83 90)
+    (property "Footprint" "xiao_256:D_DO-35_SOD27_P7.62mm_Horizontal" (at 77.47 36.83 90)
       (effects (font (size 1.27 1.27)) hide)
     )
@@
       (effects (font (size 1.27 1.27)) (justify right))
     )
-    (property "Footprint" "Diode_THT:D_DO-35_SOD27_P7.62mm_Horizontal" (at 31.75 93.98 90)
+    (property "Footprint" "xiao_256:D_DO-35_SOD27_P7.62mm_Horizontal" (at 31.75 93.98 90)
       (effects (font (size 1.27 1.27)) hide)
     )
@@
       (effects (font (size 1.27 1.27)) (justify right))
     )
-    (property "Footprint" "Diode_THT:D_DO-35_SOD27_P7.62mm_Horizontal" (at 107.95 36.83 90)
+    (property "Footprint" "xiao_256:D_DO-35_SOD27_P7.62mm_Horizontal" (at 107.95 36.83 90)
       (effects (font (size 1.27 1.27)) hide)
     )
@@
       (effects (font (size 1.27 1.27)) (justify right))
     )
-    (property "Footprint" "Diode_THT:D_DO-35_SOD27_P7.62mm_Horizontal" (at 92.71 55.88 90)
+    (property "Footprint" "xiao_256:D_DO-35_SOD27_P7.62mm_Horizontal" (at 92.71 55.88 90)
       (effects (font (size 1.27 1.27)) hide)
     )
@@
       (effects (font (size 1.27 1.27)) (justify right))
     )
-    (property "Footprint" "Diode_THT:D_DO-35_SOD27_P7.62mm_Horizontal" (at 31.75 113.03 90)
+    (property "Footprint" "xiao_256:D_DO-35_SOD27_P7.62mm_Horizontal" (at 31.75 113.03 90)
       (effects (font (size 1.27 1.27)) hide)
     )
@@
       (effects (font (size 1.27 1.27)) (justify right))
     )
-    (property "Footprint" "Diode_THT:D_DO-35_SOD27_P7.62mm_Horizontal" (at 77.47 74.93 90)
+    (property "Footprint" "xiao_256:D_DO-35_SOD27_P7.62mm_Horizontal" (at 77.47 74.93 90)
       (effects (font (size 1.27 1.27)) hide)
     )
@@
       (effects (font (size 1.27 1.27)) (justify right))
     )
-    (property "Footprint" "Diode_THT:D_DO-35_SOD27_P7.62mm_Horizontal" (at 107.95 113.03 90)
+    (property "Footprint" "xiao_256:D_DO-35_SOD27_P7.62mm_Horizontal" (at 107.95 113.03 90)
       (effects (font (size 1.27 1.27)) hide)
     )
@@
       (effects (font (size 1.27 1.27)) (justify right))
     )
-    (property "Footprint" "Diode_THT:D_DO-35_SOD27_P7.62mm_Horizontal" (at 107.95 74.93 90)
+    (property "Footprint" "xiao_256:D_DO-35_SOD27_P7.62mm_Horizontal" (at 107.95 74.93 90)
       (effects (font (size 1.27 1.27)) hide)
     )
@@
       (effects (font (size 1.27 1.27)) (justify right))
     )
-    (property "Footprint" "Diode_THT:D_DO-35_SOD27_P7.62mm_Horizontal" (at 31.75 55.88 90)
+    (property "Footprint" "xiao_256:D_DO-35_SOD27_P7.62mm_Horizontal" (at 31.75 55.88 90)
       (effects (font (size 1.27 1.27)) hide)
     )
@@
       (effects (font (size 1.27 1.27)) (justify right))
     )
-    (property "Footprint" "Diode_THT:D_DO-35_SOD27_P7.62mm_Horizontal" (at 107.95 93.98 90)
+    (property "Footprint" "xiao_256:D_DO-35_SOD27_P7.62mm_Horizontal" (at 107.95 93.98 90)
       (effects (font (size 1.27 1.27)) hide)
     )
@@
       (effects (font (size 1.27 1.27)) (justify right))
     )
-    (property "Footprint" "Diode_THT:D_DO-35_SOD27_P7.62mm_Horizontal" (at 92.71 36.83 90)
+    (property "Footprint" "xiao_256:D_DO-35_SOD27_P7.62mm_Horizontal" (at 92.71 36.83 90)
       (effects (font (size 1.27 1.27)) hide)
     )
@@
       (effects (font (size 1.27 1.27)) (justify right))
     )
-    (property "Footprint" "Diode_THT:D_DO-35_SOD27_P7.62mm_Horizontal" (at 62.23 36.83 90)
+    (property "Footprint" "xiao_256:D_DO-35_SOD27_P7.62mm_Horizontal" (at 62.23 36.83 90)
       (effects (font (size 1.27 1.27)) hide)
     )
@@
       (effects (font (size 1.27 1.27)) (justify right))
     )
-    (property "Footprint" "Diode_THT:D_DO-35_SOD27_P7.62mm_Horizontal" (at 31.75 74.93 90)
+    (property "Footprint" "xiao_256:D_DO-35_SOD27_P7.62mm_Horizontal" (at 31.75 74.93 90)
       (effects (font (size 1.27 1.27)) hide)
     )
@@
       (effects (font (size 1.27 1.27)) (justify right))
     )
-    (property "Footprint" "Diode_THT:D_DO-35_SOD27_P7.62mm_Horizontal" (at 77.47 113.03 90)
+    (property "Footprint" "xiao_256:D_DO-35_SOD27_P7.62mm_Horizontal" (at 77.47 113.03 90)
       (effects (font (size 1.27 1.27)) hide)
     )
@@
       (effects (font (size 1.27 1.27)) (justify right))
     )
-    (property "Footprint" "Diode_THT:D_DO-35_SOD27_P7.62mm_Horizontal" (at 77.47 55.88 90)
-      (effects (font (size 1.27 1.27)) hide)
-    )
+    (property "Footprint" "xiao_256:D_DO-35_SOD27_P7.62mm_Horizontal" (at 77.47 55.88 90)
+      (effects (font (size 1.27 1.27)) hide)
+    )
