File: kicad/xiao_256.kicad_pcb (KiCad board)
At the start: 2 copper layers, 137.5 x 96 mm, 70 parts, among them J1 Conn_01x02_Pin, J2 Conn_01x02_Pin, SW1 GateronLP, SW10 GateronLP, SW11 GateronLP, SW12 GateronLP, SW13 GateronLP, SW14 GateronLP, SW15 GateronLP, SW16 GateronLP, SW17 GateronLP, SW18 GateronLP, SW19 GateronLP, SW2 GateronLP, SW20 GateronLP, SW21 GateronLP, SW22 GateronLP, SW23 GateronLP, SW24 GateronLP, SW25 GateronLP, SW26 GateronLP, SW27 GateronLP, SW28 GateronLP, SW29 GateronLP, SW3 GateronLP, SW30 GateronLP, SW4 GateronLP, SW5 GateronLP, SW6 GateronLP, SW7 GateronLP, SW8 GateronLP, SW9 GateronLP, U1 Seeed XIAO, U2 SK12D07VG4

Commit message: make cover symmetric
Parts:
- moved H4 2.69 mm to (139.0, 112.5)
- moved H6 2.50 mm to (154.0, 112.5)
- moved H3 1.00 mm to (139.0, 45.5)
Changed lines of the file:
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@@
   )
   (footprint "xiao_256:Mount_M2" (layer "F.Cu")
-    (at 140 110)
+    (at 139 112.5)
     (descr "Mounting Hole 2.2mm, M2")
     (tags "mounting hole 2.2mm m2")
@@
   )
   (footprint "xiao_256:Mount_M2" (layer "F.Cu")
-    (at 140 45.5)
+    (at 139 45.5)
     (descr "Mounting Hole 2.2mm, M2")
     (tags "mounting hole 2.2mm m2")
@@
   )
   (footprint "xiao_256:Mount_M2" (layer "F.Cu")
-    (at 154 110)
+    (at 154 112.5)
     (descr "Mounting Hole 2.2mm, M2")
     (tags "mounting hole 2.2mm m2")
@@
   (gr_line (start 22 20) (end 155.5 20)
     (stroke (width 0.1) (type default)) (layer "Edge.Cuts"))
-  (gr_text "JLCJLCJLCJLC" (at 147 113.5) (layer "F.SilkS")
+  (gr_text "JLCJLCJLCJLC" (at 146.5 43.5) (layer "F.SilkS")
     (effects (font (size 1 1) (thickness 0.15)) (justify bottom))
   )
