File: kicad-cherry/xiao_256.kicad_pcb (KiCad board)
At the start: 2 copper layers, 137.5 x 96 mm, 70 parts, among them J1 Conn_01x02_Pin, J2 Conn_01x02_Pin, SW1 CherryMX, SW10 CherryMX, SW11 CherryMX, SW12 CherryMX, SW13 CherryMX, SW14 CherryMX, SW15 CherryMX, SW16 CherryMX, SW17 CherryMX, SW18 CherryMX, SW19 CherryMX, SW2 CherryMX, SW20 CherryMX, SW21 CherryMX, SW22 CherryMX, SW23 CherryMX, SW24 CherryMX, SW25 CherryMX, SW26 CherryMX, SW27 CherryMX, SW28 CherryMX, SW29 CherryMX, SW3 CherryMX, SW30 CherryMX, SW4 CherryMX, SW5 CherryMX, SW6 CherryMX, SW7 CherryMX, SW8 CherryMX, SW9 CherryMX, U1 Seeed XIAO, U2 SK12D07VG4

Commit message: finish routing cherry mx
Routing:
- net ROW5: track 109.4 -> 196.3 mm
- net ROW4: track 109.4 -> 177.2 mm
- net ROW3: track 109.4 -> 147.3 mm
- net ROW2: track 109.4 -> 125.8 mm
- net COL1: track 234.5 -> 244.0 mm
- net ROW1: track 112.0 -> 119.3 mm
- net COL2: track 216.1 -> 222.8 mm
- net COL6: track 144.5 -> 139.5 mm
- net COL3: track 197.9 -> 201.9 mm
- net COL5: track 162.3 -> 160.1 mm
- net COL4: track 179.4 -> 180.4 mm
